Commit message: Improved STL loading efficiency. STLMesh uses numpy for fast conversion of mesh.Mesh.from_file() to kivy3 Mesh object.

File: examples/urdf/RS2-7FN-Def-URDF-Exp/urdf/RS2-7FN-Def-URDF-Exp.urdf (robot description, URDF)
Before this commit: robot RS2-7FN-Def-URDF-Exp, 9 links, 8 joints
Joints:
- joint 1015-to-wrist-joint: origin xyz=-0.000149999999999901 -0.0407999999999999 0.0804868346433256 rpy=0 0 3.10225642180847 -> xyz=-0.000149999999999901 -0.0407999999999999 0.0804868346433256 rpy=0 3.1415 3.10225642180847
